File: data/schematics/chessbot.kicad_sch (KiCad schematic)
At the start: 77 parts, among them M1 Arm-Arm Servo, M2 Base-Arm Servo, M3 Body-Base Servo, M4 Gripper Servo, SW1 SW_Reed, SW10 SW_Reed, SW11 SW_Reed, SW12 SW_Reed, SW13 SW_Reed, SW14 SW_Reed, SW15 SW_Reed, SW16 SW_Reed, SW17 SW_Reed, SW18 SW_Reed, SW19 SW_Reed, SW2 SW_Reed, SW20 SW_Reed, SW21 SW_Reed, SW22 SW_Reed, SW23 SW_Reed, SW24 SW_Reed, SW25 SW_Reed, SW26 SW_Reed, SW27 SW_Reed, SW28 SW_Reed, SW29 SW_Reed, SW3 SW_Reed, SW30 SW_Reed, SW31 SW_Reed, SW32 SW_Reed, SW33 SW_Reed, SW34 SW_Reed, SW35 SW_Reed, SW36 SW_Reed, SW37 SW_Reed, SW38 SW_Reed, SW39 SW_Reed, SW4 SW_Reed, SW40 SW_Reed, SW41 SW_Reed, SW42 SW_Reed, SW43 SW_Reed, SW44 SW_Reed, SW45 SW_Reed, SW46 SW_Reed, SW47 SW_Reed, SW48 SW_Reed, SW49 SW_Reed, SW5 SW_Reed, SW50 SW_Reed, SW51 SW_Reed, SW52 SW_Reed, SW53 SW_Reed, SW54 SW_Reed, SW55 SW_Reed, SW56 SW_Reed, SW57 SW_Reed, SW58 SW_Reed, SW59 SW_Reed, SW6 SW_Reed, SW60 SW_Reed, SW61 SW_Reed, SW62 SW_Reed, SW63 SW_Reed, SW64 SW_Reed, SW7 SW_Reed, SW8 SW_Reed, SW9 SW_Reed, U1 74HC165, U2 74HC165, U3 74HC165, U4 74HC165, U5 74HC165, U6 74HC165, U7 74HC165, U8 74HC165

Commit message: Added schematics
Parts:
- added M5: Gripper Yaw, symbol Motor:Motor_Servo
Connections:
- net +6V: now also M5.2 (+)
- net at A1.6 (GND), M1.3 (-), M2.3 (-)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: now also M5.3 (-)
- net at A1.13 (SDA/A4): now also M5.1 (PWM)
Changed lines of the file:
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@@
   (junction (at 86.36 273.05) (diameter 0) (color 0 0 0 0)
   )
+  (junction (at 293.37 476.25) (diameter 0) (color 0 0 0 0)
+  )
   (junction (at 339.09 226.06) (diameter 0) (color 0 0 0 0)
   )
@@
   (junction (at 466.09 213.36) (diameter 0) (color 0 0 0 0)
   )
-  (junction (at 143.51 467.36) (diameter 0) (color 0 0 0 0)
-  )
   (junction (at 278.13 259.08) (diameter 0) (color 0 0 0 0)
   )
@@
   (junction (at 323.85 157.48) (diameter 0) (color 0 0 0 0)
   )
+  (junction (at 322.58 444.5) (diameter 0) (color 0 0 0 0)
+  )
   (junction (at 466.09 276.86) (diameter 0) (color 0 0 0 0)
   )
@@
   (junction (at 293.37 90.17) (diameter 0) (color 0 0 0 0)
   )
+  (junction (at 322.58 459.74) (diameter 0) (color 0 0 0 0)
+  )
   (junction (at 339.09 31.75) (diameter 0) (color 0 0 0 0)
   )
@@
     (stroke (width 0) (type default))
   )
-  (wire (pts (xy 293.37 444.5) (xy 293.37 485.14))
-    (stroke (width 0) (type default))
-  )
   (wire (pts (xy 54.61 157.48) (xy 54.61 223.52))
     (stroke (width 0) (type default))
@@
     (stroke (width 0) (type default))
   )
+  (wire (pts (xy 322.58 459.74) (xy 322.58 444.5))
+    (stroke (width 0) (type default))
+  )
   (wire (pts (xy 328.93 106.68) (xy 152.4 106.68))
     (stroke (width 0) (type default))
@@
     (stroke (width 0) (type default))
   )
+  (wire (pts (xy 294.64 457.2) (xy 347.98 457.2))
+    (stroke (width 0) (type default))
+  )
   (wire (pts (xy 443.23 237.49) (xy 443.23 198.12))
     (stroke (width 0) (type default))
@@
     (stroke (width 0) (type default))
   )
-  (wire (pts (xy 294.64 447.04) (xy 294.64 476.25))
+  (wire (pts (xy 293.37 447.04) (xy 293.37 476.25))
     (stroke (width 0) (type default))
   )
@@
     (stroke (width 0) (type default))
   )
-  (wire (pts (xy 294.64 476.25) (xy 265.43 476.25))
+  (wire (pts (xy 265.43 476.25) (xy 293.37 476.25))
     (stroke (width 0) (type default))
   )
@@
     (stroke (width 0) (type default))
   )
+  (wire (pts (xy 278.13 353.06) (xy 294.64 353.06))
+    (stroke (width 0) (type default))
+  )
   (wire (pts (xy 152.4 168.91) (xy 74.93 168.91))
     (stroke (width 0) (type default))
@@
     (stroke (width 0) (type default))
   )
+  (wire (pts (xy 189.23 467.36) (xy 189.23 480.06))
+    (stroke (width 0) (type default))
+  )
   (wire (pts (xy 308.61 90.17) (xy 308.61 123.19))
     (stroke (width 0) (type default))
@@
     (stroke (width 0) (type default))
   )
+  (wire (pts (xy 322.58 444.5) (xy 347.98 444.5))
+    (stroke (width 0) (type default))
+  )
   (wire (pts (xy 506.73 121.92) (xy 534.67 121.92))
     (stroke (width 0) (type default))
@@
     (stroke (width 0) (type default))
   )
+  (wire (pts (xy 194.31 467.36) (xy 189.23 467.36))
+    (stroke (width 0) (type default))
+  )
   (wire (pts (xy 440.69 317.5) (xy 481.33 317.5))
     (stroke (width 0) (type default))
@@
     (stroke (width 0) (type default))
   )
+  (wire (pts (xy 322.58 459.74) (xy 347.98 459.74))
+    (stroke (width 0) (type default))
+  )
   (wire (pts (xy 59.69 109.22) (xy 59.69 175.26))
     (stroke (width 0) (type default))
@@
     (stroke (width 0) (type default))
   )
-  (wire (pts (xy 143.51 443.23) (xy 143.51 467.36))
-    (stroke (width 0) (type default))
-  )
   (wire (pts (xy 86.36 273.05) (xy 86.36 349.25))
     (stroke (width 0) (type default))
@@
     (stroke (width 0) (type default))
   )
+  (wire (pts (xy 293.37 476.25) (xy 344.17 476.25))
+    (stroke (width 0) (type default))
+  )
   (wire (pts (xy 320.04 398.78) (xy 234.95 398.78))
     (stroke (width 0) (type default))
@@
     (stroke (width 0) (type default))
   )
+  (wire (pts (xy 344.17 462.28) (xy 344.17 476.25))
+    (stroke (width 0) (type default))
+  )
   (wire (pts (xy 421.64 127) (xy 481.33 127))
     (stroke (width 0) (type default))
@@
     (stroke (width 0) (type default))
   )
+  (wire (pts (xy 294.64 353.06) (xy 294.64 457.2))
+    (stroke (width 0) (type default))
+  )
   (wire (pts (xy 494.03 223.52) (xy 519.43 223.52))
     (stroke (width 0) (type default))
@@
     (stroke (width 0) (type default))
   )
-  (wire (pts (xy 347.98 444.5) (xy 293.37 444.5))
-    (stroke (width 0) (type default))
-  )
   (wire (pts (xy 134.62 185.42) (xy 134.62 337.82))
     (stroke (width 0) (type default))
@@
     (stroke (width 0) (type default))
   )
+  (wire (pts (xy 322.58 421.64) (xy 322.58 444.5))
+    (stroke (width 0) (type default))
+  )
   (wire (pts (xy 419.1 196.85) (xy 419.1 121.92))
     (stroke (width 0) (type default))
@@
     (stroke (width 0) (type default))
   )
-  (wire (pts (xy 293.37 485.14) (xy 143.51 485.14))
-    (stroke (width 0) (type default))
-  )
   (wire (pts (xy 267.97 96.52) (xy 147.32 96.52))
     (stroke (width 0) (type default))
@@
     (stroke (width 0) (type default))
   )
-  (wire (pts (xy 143.51 467.36) (xy 143.51 485.14))
-    (stroke (width 0) (type default))
-  )
   (wire (pts (xy 313.69 298.45) (xy 440.69 298.45))
     (stroke (width 0) (type default))
@@
     (stroke (width 0) (type default))
   )
+  (wire (pts (xy 347.98 462.28) (xy 344.17 462.28))
+    (stroke (width 0) (type default))
+  )
   (wire (pts (xy 270.51 294.64) (xy 494.03 294.64))
     (stroke (width 0) (type default))
@@
     (stroke (width 0) (type default))
   )
-  (wire (pts (xy 143.51 467.36) (xy 194.31 467.36))
-    (stroke (width 0) (type default))
-  )
   (wire (pts (xy 59.69 175.26) (xy 59.69 240.03))
     (stroke (width 0) (type default))
@@
     (stroke (width 0) (type default))
   )
+  (wire (pts (xy 322.58 480.06) (xy 322.58 459.74))
+    (stroke (width 0) (type default))
+  )
   (wire (pts (xy 481.33 149.86) (xy 466.09 149.86))
     (stroke (width 0) (type default))
@@
     (stroke (width 0) (type default))
   )
+  (wire (pts (xy 189.23 480.06) (xy 322.58 480.06))
+    (stroke (width 0) (type default))
+  )
   (wire (pts (xy 344.17 175.26) (xy 194.31 175.26))
     (stroke (width 0) (type default))
@@
     (stroke (width 0) (type default))
   )
-  (wire (pts (xy 347.98 447.04) (xy 294.64 447.04))
+  (wire (pts (xy 347.98 447.04) (xy 293.37 447.04))
     (stroke (width 0) (type default))
   )
@@
         (path "/3a094df6-8261-4de4-8a7c-d317b8c4e0e5"
           (reference "SW8") (unit 1)
+        )
+      )
+    )
+  )
+  (symbol (lib_id "power:+6V") (at 322.58 421.64 0) (unit 1)
+    (in_bom yes) (on_board yes) (dnp no) (fields_autoplaced)
+    (property "Reference" "#PWR03" (at 322.58 425.45 0)
+      (effects (font (size 1.27 1.27)) hide)
+    )
+    (property "Value" "+6V" (at 322.58 416.56 0)
+      (effects (font (size 1.27 1.27)))
+    )
+    (property "Footprint" "" (at 322.58 421.64 0)
+      (effects (font (size 1.27 1.27)) hide)
+    )
+    (property "Datasheet" "" (at 322.58 421.64 0)
+      (effects (font (size 1.27 1.27)) hide)
+    )
+    (pin "1")
+    (instances
+      (project "chessbot"
+        (path "/3a094df6-8261-4de4-8a7c-d317b8c4e0e5"
+          (reference "#PWR03") (unit 1)
         )
       )
@@
         )
       )
+    )
+  )
+  (symbol (lib_id "Motor:Motor_Servo") (at 355.6 459.74 0) (unit 1)
+    (in_bom yes) (on_board yes) (dnp no) (fields_autoplaced)
+    (property "Reference" "M5" (at 364.49 458.0366 0)
+      (effects (font (size 1.27 1.27)) (justify left))
+    )
+    (property "Value" "Gripper Yaw" (at 364.49 460.5766 0)
+      (effects (font (size 1.27 1.27)) (justify left))
+    )
+    (property "Footprint" "" (at 355.6 464.566 0)
+      (effects (font (size 1.27 1.27)) hide)
+    )
+    (property "Datasheet" "http://forums.parallax.com/uploads/attachments/46831/74481.png" (at 355.6 464.566 0)
+      (effects (font (size 1.27 1.27)) hide)
+    )
+    (pin "1")
+    (pin "2")
+    (pin "3")
+    (instances
+      (project "chessbot"
+        (path "/3a094df6-8261-4de4-8a7c-d317b8c4e0e5"
+          (reference "M5") (unit 1)
+        )
+      )
